File: Autoflate_HW.kicad_sch (KiCad schematic)
At the start: 69 parts, among them J1 JST_XH_3, J10 JST_VH_2, J11 JST_VH_2, J12 JST_XH_3, J13 Header_1, J2 JST_VH_3, J3 Conn_01x04_Male, J6 JST_XH_4, J7 Header_2, J8 Header_4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

Commit message: Generated schematic pdf
Other:
- company: (none) -> Ran Katz
- title: (none) -> Autoflate - Tire inflator controller board
Changed lines of the file:
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@@
 (kicad_sch (version 20211123) (generator eeschema)
   (paper "A4")
+  (title_block
+    (title "Autoflate - Tire inflator controller board")
+    (date "2022-09-15")
+    (rev "1.0")
+    (company "Ran Katz")
+  )
   (junction (at 250.19 118.11) (diameter 0) (color 0 0 0 0)
   )
